Commit message: Urdf coordination space update

File: urdf/PhoXi3Dscanner_values.xacro (robot description, xacro)
@@ -1,7 +1,15 @@
 <?xml version="1.0" ?>
 <robot xmlns:xacro="http://ros.org/wiki/xacro">
+    <!--PhoXi3Dscanner XS old-->
+    <xacro:macro name="PhoXi3DscannerXS_old_default_sensor_origin">
+        <origin xyz="0.1 0.025 0.035" rpy="0 ${-15.45/180*pi} ${pi}" />
+    </xacro:macro>
+    <xacro:macro name="PhoXi3DscannerXS_old_meshes">
+        <mesh filename="package://phoxi_camera/meshes/visual/PhoXi_XS_old.f.STL" scale = "0.001 0.001 0.001"/>
+        <mesh filename="package://phoxi_camera/meshes/collision/PhoXi_XS_old.c.STL" scale = "0.001 0.001 0.001"/>
+    </xacro:macro>
     <!--PhoXi3Dscanner XS-->
     <xacro:macro name="PhoXi3DscannerXS_default_sensor_origin">
-        <origin xyz="0.1 0.025 0.035" rpy="0 -0.26965337 0" />
+        <origin xyz="0.090 0.0299 0.03595" rpy="0 ${0/180*pi} ${pi}" />
     </xacro:macro>
     <xacro:macro name="PhoXi3DscannerXS_meshes">
@@ -11,5 +19,5 @@
     <!--PhoXi3Dscanner S-->
     <xacro:macro name="PhoXi3DscannerS_default_sensor_origin">
-        <origin xyz="${0.23 / 2.0} 0.0168 0.035" rpy="0 -0.26965337 0" />
+        <origin xyz="-0.1173845315 0.0299 0.005287752939" rpy="0 ${-15.45/180*pi} ${pi}" />
     </xacro:macro>
     <xacro:macro name="PhoXi3DscannerS_meshes">
@@ -19,5 +27,5 @@
     <!--PhoXi3Dscanner M-->
     <xacro:macro name="PhoXi3DscannerM_default_sensor_origin">
-        <origin xyz="${0.350 / 2.0} 0.0168 0.035" rpy="0 -0.20507619 0" />
+        <origin xyz="-0.176277236938477 0.0299 0.002164826095" rpy="0 ${-11.75/180*pi} ${pi}" />
     </xacro:macro>
     <xacro:macro name="PhoXi3DscannerM_meshes">
@@ -27,5 +35,5 @@
     <!--PhoXi3Dscanner L-->
     <xacro:macro name="PhoXi3DscannerL_default_sensor_origin">
-        <origin xyz="${(0.55 / 2.0)} 0.0168 0.035" rpy="0 -0.1649336 0" />
+        <origin xyz="-0.274213 0.0299 0.0090044" rpy="0 ${-9.45/180*pi} ${pi}" />
     </xacro:macro>
     <xacro:macro name="PhoXi3DscannerL_meshes">
@@ -35,5 +43,5 @@
     <!--PhoXi3Dscanner XL-->
     <xacro:macro name="PhoXi3DscannerXL_default_sensor_origin">
-        <origin xyz="${0.850 / 2.0} 0.0168 0.035" rpy="0 -0.1309 0" />
+        <origin xyz="-0.4349977156 0.0299 0.02086702926" rpy="0 ${-7.5/180*pi} ${pi}" />
     </xacro:macro>
     <xacro:macro name="PhoXi3DscannerXL_meshes">
